File: 2-Hardware/design/Crane_Interface.kicad_pcb (KiCad board)
At the start: 2 copper layers, 81.3 x 31.8 mm, 6 parts, among them J1 PMOD_DUAL, J2 PMOD_DUAL, J3 PMOD_DUAL, J4 PMOD_DUAL, P1 CONN_040, P2 CONN_003

Commit message: Board design
Parts:
- added P3: CONN_006, Connectors:CONN_2.54mm_2x03, F.Cu at (161.3, 95.2)
- moved P2 6.48 mm to (118.7, 95.2), turned to 180 degrees
Connections:
- net /DIO18 renamed /Y_PWM
- J1 pad 1: /DIO0 -> /AX_ENC_A
- J1 pad 10: /DIO7 -> Net-(J1-Pad10)
- J1 pad 12: VCC -> Net-(J1-Pad12)
- J1 pad 2: /DIO2 -> /AX_ENC_B
- J1 pad 3: /DIO4 -> /AY_ENC_A
- J1 pad 4: /DIO6 -> /AY_ENC_B
- J1 pad 6: VCC -> Net-(J1-Pad6)
- J1 pad 7: /DIO1 -> Net-(J1-Pad7)
- J1 pad 8: /DIO3 -> Net-(J1-Pad8)
- J1 pad 9: /DIO5 -> Net-(J1-Pad9)
- J2 pad 1: /DIO8 -> /Z_THERM
- J2 pad 10: /DIO15 -> Net-(J2-Pad10)
- J2 pad 12: VCC -> Net-(J2-Pad12)
- J2 pad 2: /DIO10 -> /Z_PWM
- J2 pad 3: /DIO12 -> /Z_BRAKE
- J2 pad 4: /DIO14 -> /Z_DIR
- J2 pad 6: VCC -> Net-(J2-Pad6)
- J2 pad 7: /DIO9 -> /Z_ENC_B
- J2 pad 8: /DIO11 -> /Z_ENC_A
- J2 pad 9: /DIO13 -> /Z_SWITCH
- J3 pad 1: /DIO16 -> /Y_THERM
- J3 pad 10: /DIO23 -> Net-(J3-Pad10)
- J3 pad 12: VCC -> Net-(J3-Pad12)
- J3 pad 3: /DIO20 -> /Y_BRAKE
- J3 pad 4: /DIO22 -> /Y_DIR
- J3 pad 6: VCC -> Net-(J3-Pad6)
- J3 pad 7: /DIO17 -> /Y_ENC_B
- J3 pad 8: /DIO19 -> /Y_ENC_A
- J3 pad 9: /DIO21 -> /Y_SWITCH
- J4 pad 1: /DIO24 -> /X_THERM
- J4 pad 2: /DIO25 -> /X_PWM
- J4 pad 3: Net-(J4-Pad3) -> /X_BRAKE
- J4 pad 4: Net-(J4-Pad4) -> /X_DIR
- J4 pad 7: Net-(J4-Pad7) -> /X_ENC_B
- J4 pad 8: Net-(J4-Pad8) -> /X_ENC_A
- J4 pad 9: Net-(J4-Pad9) -> /X_SWITCH
- P1 pad 1: /DIO0 -> /X_ENC_A
- P1 pad 11: /DIO5 -> /AX_ENC_B
- P1 pad 13: /DIO6 -> /AY_ENC_A
- P1 pad 15: /DIO7 -> /AY_ENC_B
- P1 pad 17: /DIO8 -> /Z_ENC_A_USB
- P1 pad 19: /DIO9 -> /Z_ENC_B_USB
- P1 pad 2: GND -> /Z_ENC_A_PCI
- P1 pad 21: /DIO10 -> /Z_SWITCH
- P1 pad 22: /DIO11 -> /X_SWITCH
- P1 pad 23: /DIO12 -> /Y_SWITCH
- P1 pad 24: /DIO13 -> /Z_THERM
- P1 pad 25: /DIO14 -> /Z_PWM
- P1 pad 26: /DIO15 -> /Z_BRAKE
- P1 pad 27: /DIO16 -> /Z_DIR
- P1 pad 28: /DIO17 -> /Y_THERM
- P1 pad 3: /DIO1 -> /X_ENC_B
- P1 pad 30: /DIO19 -> /Y_BRAKE
- P1 pad 31: /DIO20 -> /Y_DIR
- P1 pad 32: /DIO21 -> /X_THERM
- P1 pad 33: /DIO22 -> /X_PWM
- P1 pad 34: /DIO23 -> /X_BRAKE
- P1 pad 35: /DIO24 -> /X_DIR
- P1 pad 36: /DIO25 -> GND
- P1 pad 4: GND -> /Z_ENC_B_PCI
- P1 pad 5: /DIO2 -> /Y_ENC_A
- P1 pad 7: /DIO3 -> /Y_ENC_B
- P1 pad 9: /DIO4 -> /AX_ENC_A
Routing:
- net VCC: track 106.7 -> 24.5 mm
- net /X_ENC_A: track 0.00 -> 72.3 mm
- net /X_ENC_B: track 0.00 -> 67.1 mm
- net /X_SWITCH: track 0.00 -> 50.4 mm, vias 0 -> 2
- net /Y_ENC_A: track 0.00 -> 48.4 mm, vias 0 -> 1
- net /Y_ENC_B: track 0.00 -> 44.8 mm, vias 0 -> 1
- net /Z_THERM: track 0.00 -> 40.4 mm, vias 0 -> 2
- net /AX_ENC_A: track 0.00 -> 38.6 mm, vias 0 -> 1
- net /Z_BRAKE: track 0.00 -> 38.5 mm, vias 0 -> 2
- net /AX_ENC_B: track 0.00 -> 38.3 mm, vias 0 -> 1
- net /AY_ENC_A: track 0.00 -> 37.9 mm, vias 0 -> 1
- net /AY_ENC_B: track 0.00 -> 37.5 mm, vias 0 -> 1
- net /DIO7: track 37.4 -> 0.00 mm
- net /Z_PWM: track 0.00 -> 36.1 mm, vias 0 -> 2
- net /DIO5: track 35.7 -> 0.00 mm
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Other:
- board text added: "PCI"
- board text added: "PMOD-Compatible Interface for the InTeCo Crane"
- board text added: "USB"
- board text removed: "PMOD Compatible Interface for the 40-pin InTeCo Connector"

Commit message: Added silkscreen label
Other:
- board text added: "Designed by Ian McInerney"
Changed lines of the file:
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@@
     (links 51)
     (no_connects 0)
-    (area 106.604999 79.934999 188.035001 111.835001)
+    (area 106.404999 79.734999 188.235001 111.835001)
     (thickness 1.6)
-    (drawings 9)
+    (drawings 10)
     (tracks 214)
     (zones 0)
@@
       (net 22 /Z_ENC_A_USB))
   )
+  (gr_text "Designed by Ian McInerney" (at 147.32 109.22) (layer B.SilkS)
+    (effects (font (size 1.5 1.5) (thickness 0.3)) (justify mirror))
+  )
   (gr_text USB (at 156.21 95.25 270) (layer F.SilkS)
