File: 2-Hardware/design/Crane_Interface.sch (KiCad schematic (older format))
At the start: 5 parts, among them J1 PMOD_DUAL, J2 PMOD_DUAL, J3 PMOD_DUAL, J4 PMOD_DUAL, P1 CONN_040

Commit message: Initial design
* Renamed design
* Initial schematic and board layout
Parts:
- added P2: CONN_003, Connectors:CONN_2.54mm_1x03, symbol CONN_003
Connections:
- net +3V3: now also P2.1; no longer J1.12 (VCC), J1.6 (VCC), J2.12 (VCC), J2.6 (VCC), J3.12 (VCC), J3.6 (VCC), J4.12 (VCC), J4.6 (VCC)
- net +5V: now also P2.3
- net DIO0: now also J1.1 (IO1_1)
- net DIO1: now also J1.7 (IO2_1)
- net DIO10: now also J2.2 (IO1_2)
- net DIO11: now also J2.8 (IO2_2)
- net DIO12: now also J2.3 (IO1_3)
- net DIO13: now also J2.9 (IO2_3)
- net DIO14: now also J2.4 (IO1_4)
- net DIO15: now also J2.10 (IO2_4)
- net DIO16: now also J3.1 (IO1_1)
- net DIO17: now also J3.7 (IO2_1)
- net DIO18: now also J3.2 (IO1_2)
- net DIO19: now also J3.8 (IO2_2)
- net DIO2: now also J1.2 (IO1_2)
- net DIO20: now also J3.3 (IO1_3)
- net DIO21: now also J3.9 (IO2_3)
- net DIO22: now also J3.4 (IO1_4)
- net DIO23: now also J3.10 (IO2_4)
- net DIO24: now also J4.1 (IO1_1)
- net DIO25: now also J4.2 (IO1_2)
- net DIO3: now also J1.8 (IO2_2)
- net DIO4: now also J1.3 (IO1_3)
- net DIO5: now also J1.9 (IO2_3)
- net DIO6: now also J1.4 (IO1_4)
- net DIO7: now also J1.10 (IO2_4)
- net DIO8: now also J2.1 (IO1_1)
- net DIO9: now also J2.7 (IO2_1)
- new net VCC: J1.12 (VCC), J1.6 (VCC), J2.12 (VCC), J2.6 (VCC), J3.12 (VCC), J3.6 (VCC), J4.12 (VCC), J4.6 (VCC), P2.2
Other:
- note added: "Voltage Selector"
- moved on the sheet: J1B, J1C, J2B, J2C, J3B, J3C, J4B, J4C

Commit message: Board design
Parts:
- added P3: CONN_006, Connectors:CONN_2.54mm_2x03, symbol CONN_006
Connections:
- net GND: now also P1.36; no longer P1.2, P1.4
- net VCC: no longer J1.12 (VCC), J1.6 (VCC), J2.12 (VCC), J2.6 (VCC), J3.12 (VCC), J3.6 (VCC)
- net X_BRAKE: now reaches J4.3 (IO1_3)
- net X_BRAKE: now also P1.34
- net X_DIR: now reaches J4.4 (IO1_4)
- net X_DIR: now also P1.35
- net X_ENC_B: now reaches J4.7 (IO2_1)
- net X_ENC_B: now also P1.3
- net X_ENC_A: now reaches J4.8 (IO2_2)
- net X_ENC_A: now also P1.1
- net X_SWITCH: now reaches J4.9 (IO2_3)
- net X_SWITCH: now also P1.22
- net DIO0 renamed AX_ENC_A
- net AX_ENC_A: now also P1.9; no longer P1.1
- net DIO1: no longer names the net of J1.7 (IO2_1)
- net DIO1: no longer P1.3
- net DIO10 renamed Z_PWM
- net Z_PWM: now also P1.25; no longer P1.21
- net DIO11 renamed Z_ENC_A
- net Z_ENC_A: now also P3.4; no longer P1.22
- net DIO12 renamed Y_SWITCH
- net Y_SWITCH: now also J3.9 (IO2_3); no longer J2.3 (IO1_3)
- net DIO13 renamed Z_SWITCH
- net Z_SWITCH: now also P1.21; no longer P1.24
- net DIO14 renamed Z_DIR
- net Z_DIR: now also P1.27; no longer P1.25
- net DIO15: no longer names the net of J2.10 (IO2_4)
- net DIO15: no longer P1.26
- net DIO16 renamed Y_THERM
- net Y_THERM: now also P1.28; no longer P1.27
- net DIO17 renamed Y_ENC_B
- net Y_ENC_B: now also P1.7; no longer P1.28
- net DIO18 renamed Y_PWM
- net DIO19 renamed Y_BRAKE
- net Y_BRAKE: now also J3.3 (IO1_3); no longer J3.8 (IO2_2)
- net DIO2 renamed AX_ENC_B
- net AX_ENC_B: now also P1.11; no longer P1.5
- net DIO20 renamed Y_DIR
- net Y_DIR: now also J3.4 (IO1_4); no longer J3.3 (IO1_3)
- net DIO21 renamed X_THERM
- net X_THERM: now also J4.1 (IO1_1); no longer J3.9 (IO2_3)
- net DIO22 renamed X_PWM
- net X_PWM: now also J4.2 (IO1_2); no longer J3.4 (IO1_4)
- net DIO23: no longer names the net of J3.10 (IO2_4)
- net DIO23: no longer P1.34
- removed net DIO24: J4.1 (IO1_1), P1.35
- removed net DIO25: J4.2 (IO1_2), P1.36
- net DIO3: no longer names the net of J1.8 (IO2_2)
- net DIO3: no longer P1.7
- net DIO4 renamed AY_ENC_A
- net AY_ENC_A: now also P1.13; no longer P1.9
- net DIO5: no longer names the net of J1.9 (IO2_3)
- net DIO5: no longer P1.11
- net DIO6 renamed AY_ENC_B
- net AY_ENC_B: now also P1.15; no longer P1.13
- net DIO7: no longer names the net of J1.10 (IO2_4)
- net DIO7: no longer P1.15
- net DIO8 renamed Z_ENC_A_USB
- net Z_ENC_A_USB: now also P3.6; no longer J2.1 (IO1_1)
- net DIO9 renamed Z_ENC_B
- net Z_ENC_B: now also P3.3; no longer P1.19
- new net Y_ENC_A: J3.8 (IO2_2), P1.5
- new net Z_BRAKE: J2.3 (IO1_3), P1.26
- new net Z_ENC_A_PCI: P1.2, P3.2
- new net Z_ENC_B_PCI: P1.4, P3.1
- new net Z_ENC_B_USB: P1.19, P3.5
- new net Z_THERM: J2.1 (IO1_1), P1.24
Changed lines of the file:
@@
 Connection ~ 1300 4450
-Wire Wire Line
-	1300 1050 1300 1200
-Wire Wire Line
-	1300 1100 1200 1100
-Wire Wire Line
-	1300 1200 1200 1200
-Connection ~ 1300 1100
 Wire Wire Line
 	1200 1400 1300 1400
@@
 Connection ~ 1300 1500
 Wire Wire Line
-	1300 2200 1200 2200
-Wire Wire Line
-	1300 2050 1300 2200
-Wire Wire Line
-	1200 2100 1300 2100
-Connection ~ 1300 2100
-Wire Wire Line
 	1200 2500 1300 2500
 Wire Wire Line
@@
 	1200 2400 1300 2400
 Connection ~ 1300 2500
-Wire Wire Line
-	1300 3200 1200 3200
-Wire Wire Line
-	1300 3050 1300 3200
-Wire Wire Line
-	1200 3100 1300 3100
-Connection ~ 1300 3100
 Wire Wire Line
 	1200 3400 1300 3400
@@
 	1    0    0    -1
 $EndComp
-Wire Wire Line
-	8300 1350 8400 1350
-Wire Wire Line
-	8400 1350 8400 2650
-Wire Wire Line
-	8300 1650 8400 1650
-Connection ~ 8400 1650
-Wire Wire Line
-	8300 1950 8400 1950
-Connection ~ 8400 1950
-Wire Wire Line
-	8300 2250 8400 2250
-Connection ~ 8400 2250
-Wire Wire Line
-	8300 2550 8400 2550
-Connection ~ 8400 2550
 $Comp
 L GND #PWR07
@@
 $EndComp
 Wire Wire Line
-	9950 3900 9950 4450
+	9950 3750 9950 4450
 Wire Wire Line
 	9950 4050 9750 4050
@@
 Connection ~ 9950 4050
 Text Label 8450 1200 0    60   ~ 0
-DIO0
+X_ENC_A
 Text Label 8450 1500 0    60   ~ 0
-DIO1
+X_ENC_B
 Text Label 8450 1800 0    60   ~ 0
-DIO2
+Y_ENC_A
 Text Label 8450 2100 0    60   ~ 0
-DIO3
+Y_ENC_B
 Text Label 8450 2400 0    60   ~ 0
-DIO4
+AX_ENC_A
 Wire Wire Line
 	8450 2400 8300 2400
@@
 	8300 1200 8450 1200
 Text Label 8450 2950 0    60   ~ 0
-DIO5
+AX_ENC_B
 Text Label 8450 3250 0    60   ~ 0
-DIO6
+AY_ENC_A
 Text Label 8450 3550 0    60   ~ 0
-DIO7
+AY_ENC_B
 Text Label 8450 3850 0    60   ~ 0
-DIO8
+Z_ENC_A_USB
 Text Label 8450 4150 0    60   ~ 0
-DIO9
+Z_ENC_B_USB
 Text Label 9900 1250 0    60   ~ 0
-DIO10
+Z_SWITCH
 Text Label 9900 1400 0    60   ~ 0
-DIO11
+X_SWITCH
 Text Label 9900 1550 0    60   ~ 0
-DIO12
+Y_SWITCH
 Text Label 9900 1700 0    60   ~ 0
-DIO13
+Z_THERM
 Text Label 9900 1850 0    60   ~ 0
-DIO14
+Z_PWM
 Text Label 9900 2000 0    60   ~ 0
-DIO15
+Z_BRAKE
 Text Label 9900 2150 0    60   ~ 0
-DIO16
+Z_DIR
 Text Label 9900 2300 0    60   ~ 0
-DIO17
+Y_THERM
 Text Label 9900 2450 0    60   ~ 0
-DIO18
+Y_PWM
 Text Label 9900 2600 0    60   ~ 0
-DIO19
+Y_BRAKE
 Text Label 9900 3000 0    60   ~ 0
-DIO20
+Y_DIR
 Text Label 9900 3150 0    60   ~ 0
-DIO21
+X_THERM
 Text Label 9900 3300 0    60   ~ 0
-DIO22
+X_PWM
 Text Label 9900 3450 0    60   ~ 0
-DIO23
+X_BRAKE
 Text Label 9900 3600 0    60   ~ 0
-DIO24
-Text Label 9900 3750 0    60   ~ 0
-DIO25
+X_DIR
 Wire Wire Line
 	8450 2950 8300 2950
@@
 	9900 3600 9750 3600
 Wire Wire Line
-	9750 3750 9900 3750
+	9750 3750 9950 3750
 Text Notes 8750 800  0    60   ~ 0
 Crane Connector
@@
 Text Notes 5800 700  0    60   ~ 0
 PMOD 4
-Text Label 2850 1150 0    60   ~ 0
-DIO0
-Text Label 2850 2100 0    60   ~ 0
-DIO1
-Text Label 2850 1250 0    60   ~ 0
-DIO2
-Text Label 2850 2200 0    60   ~ 0
-DIO3
-Text Label 2850 1350 0    60   ~ 0
-DIO4
-Text Label 2850 2300 0    60   ~ 0
-DIO5
-Text Label 2850 1450 0    60   ~ 0
-DIO6
-Text Label 2850 2400 0    60   ~ 0
-DIO7
-Text Label 4000 1150 0    60   ~ 0
-DIO8
-Text Label 4000 2150 0    60   ~ 0
-DIO9
-Text Label 4000 1250 0    60   ~ 0
-DIO10
-Text Label 4000 2250 0    60   ~ 0
-DIO11
-Text Label 4000 1350 0    60   ~ 0
-DIO12
-Text Label 4000 2350 0    60   ~ 0
-DIO13
-Text Label 4000 1450 0    60   ~ 0
-DIO14
-Text Label 4000 2450 0    60   ~ 0
-DIO15
-Text Label 5150 1150 0    60   ~ 0
-DIO16
-Text Label 5150 2150 0    60   ~ 0
-DIO17
-Text Label 5150 1250 0    60   ~ 0
-DIO18
-Text Label 5150 2250 0    60   ~ 0
-DIO19
-Text Label 5150 1350 0    60   ~ 0
-DIO20
-Text Label 5150 2350 0    60   ~ 0
-DIO21
-Text Label 5150 1450 0    60   ~ 0
-DIO22
-Text Label 5150 2450 0    60   ~ 0
-DIO23
-Text Label 6300 1150 0    60   ~ 0
-DIO24
-Text Label 6300 1250 0    60   ~ 0
-DIO25
-Wire Wire Line
-	2750 1150 2850 1150
-Wire Wire Line
-	2850 1250 2750 1250
-Wire Wire Line
-	2750 1350 2850 1350
-Wire Wire Line
-	2850 1450 2750 1450
-Wire Wire Line
-	2750 2100 2850 2100
-Wire Wire Line
-	2850 2200 2750 2200
-Wire Wire Line
-	2750 2300 2850 2300
-Wire Wire Line
-	2850 2400 2750 2400
-Wire Wire Line
-	3900 2450 4000 2450
-Wire Wire Line
-	4000 2350 3900 2350
-Wire Wire Line
-	3900 2250 4000 2250
-Wire Wire Line
-	4000 2150 3900 2150
-Wire Wire Line
-	3900 1450 4000 1450
-Wire Wire Line
-	4000 1350 3900 1350
-Wire Wire Line
-	3900 1250 4000 1250
-Wire Wire Line
-	4000 1150 3900 1150
-Wire Wire Line
-	5050 1150 5150 1150
-Wire Wire Line
-	5150 1250 5050 1250
-Wire Wire Line
-	5050 1350 5150 1350
-Wire Wire Line
-	5150 1450 5050 1450
-Wire Wire Line
-	5050 2150 5150 2150
-Wire Wire Line
-	5150 2250 5050 2250
-Wire Wire Line
-	5050 2350 5150 2350
-Wire Wire Line
-	5150 2450 5050 2450
-Wire Wire Line
-	6300 1150 6200 1150
-Wire Wire Line
-	6200 1250 6300 1250
 $Comp
 L VCC #PWR010
@@
 $EndComp
 $Comp
-L VCC #PWR011
-U 1 1 5BB4C595
-P 1300 3050
-F 0 "#PWR011" H 1300 2900 50  0001 C CNN
-F 1 "VCC" H 1300 3200 50  0000 C CNN
-F 2 "" H 1300 3050 50  0000 C CNN
-F 3 "" H 1300 3050 50  0000 C CNN
-	1    1300 3050
-	1    0    0    -1
-$EndComp
-$Comp
-L VCC #PWR012
-U 1 1 5BB4C5EA
-P 1300 2050
-F 0 "#PWR012" H 1300 1900 50  0001 C CNN
-F 1 "VCC" H 1300 2200 50  0000 C CNN
-F 2 "" H 1300 2050 50  0000 C CNN
-F 3 "" H 1300 2050 50  0000 C CNN
-	1    1300 2050
-	1    0    0    -1
-$EndComp
-$Comp
-L VCC #PWR013
-U 1 1 5BB4C66F
-P 1300 1050
-F 0 "#PWR013" H 1300 900 50  0001 C CNN
-F 1 "VCC" H 1300 1200 50  0000 C CNN
-F 2 "" H 1300 1050 50  0000 C CNN
-F 3 "" H 1300 1050 50  0000 C CNN
-	1    1300 1050
-	1    0    0    -1
-$EndComp
-$Comp
 L CONN_003 P2
 U 1 1 5BB4C9D8
@@
 Wire Notes Line
 	1600 6050 500  6050
+Text Label 8450 1350 0    60   ~ 0
+Z_ENC_A_PCI
+Text Label 8450 1650 0    60   ~ 0
+Z_ENC_B_PCI
+Wire Wire Line
+	8300 1350 8450 1350
+Wire Wire Line
+	8450 1650 8300 1650
+Wire Wire Line
+	8300 1950 8400 1950
+Wire Wire Line
+	8400 1950 8400 2650
+Wire Wire Line
+	8300 2250 8400 2250
+Connection ~ 8400 2250
+Wire Wire Line
+	8300 2550 8400 2550
+Connection ~ 8400 2550
+Connection ~ 9950 3900
+Text Label 2800 5200 0    60   ~ 0
+Z_ENC_A_PCI
+Text Label 2800 5800 0    60   ~ 0
+Z_ENC_A_USB
+Text Label 2800 5500 0    60   ~ 0
+Z_ENC_A
+Text Label 2800 5050 0    60   ~ 0
+Z_ENC_B_PCI
+Text Label 2800 5350 0    60   ~ 0
+Z_ENC_B
+Text Label 2800 5650 0    60   ~ 0
+Z_ENC_B_USB
+Text Label 6300 2250 0    60   ~ 0
+X_ENC_A
+Text Label 6300 2150 0    60   ~ 0
+X_ENC_B
+Text Label 5150 2250 0    60   ~ 0
+Y_ENC_A
+Text Label 5150 2150 0    60   ~ 0
+Y_ENC_B
+Text Label 2850 1150 0    60   ~ 0
+AX_ENC_A
+Text Label 2850 1250 0    60   ~ 0
+AX_ENC_B
+Text Label 2850 1350 0    60   ~ 0
+AY_ENC_A
+Text Label 2850 1450 0    60   ~ 0
+AY_ENC_B
+$Comp
+L CONN_006 P3
+U 1 1 5BB50392
+P 2500 5400
+F 0 "P3" H 2500 5850 60  0000 C CNN
+F 1 "CONN_006" H 2500 4900 60  0000 C CNN
+F 2 "Connectors:CONN_2.54mm_2x03" H 2500 5450 60  0001 C CNN
+F 3 "" H 2500 5450 60  0000 C CNN
+	1    2500 5400
+	1    0    0    -1
+$EndComp
+Wire Wire Line
+	2800 5050 2700 5050
+Wire Wire Line
+	2700 5200 2800 5200
+Wire Wire Line
+	2800 5350 2700 5350
+Wire Wire Line
+	2700 5500 2800 5500
+Wire Wire Line
+	2800 5650 2700 5650
+Wire Wire Line
+	2700 5800 2800 5800
+Text Label 6300 2350 0    60   ~ 0
+X_SWITCH
+Text Label 6300 1150 0    60   ~ 0
+X_THERM
+Text Label 6300 1250 0    60   ~ 0
+X_PWM
+Text Label 6300 1450 0    60   ~ 0
+X_DIR
+Text Label 6300 1350 0    60   ~ 0
+X_BRAKE
+Text Label 5150 2350 0    60   ~ 0
+Y_SWITCH
+Text Label 5150 1150 0    60   ~ 0
+Y_THERM
+Text Label 5150 1250 0    60   ~ 0
+Y_PWM
+Text Label 5150 1450 0    60   ~ 0
+Y_DIR
+Text Label 5150 1350 0    60   ~ 0
+Y_BRAKE
+Text Label 4000 1250 0    60   ~ 0
+Z_PWM
+Text Label 4000 1450 0    60   ~ 0
+Z_DIR
+Text Label 4000 1350 0    60   ~ 0
+Z_BRAKE
+Text Label 4000 1150 0    60   ~ 0
+Z_THERM
+Text Label 4000 2250 0    60   ~ 0
+Z_ENC_A
+Text Label 4000 2150 0    60   ~ 0
+Z_ENC_B
+Text Label 4000 2350 0    60   ~ 0
+Z_SWITCH
+Wire Wire Line
+	2750 1150 2850 1150
+Wire Wire Line
+	2850 1250 2750 1250
+Wire Wire Line
+	2750 1350 2850 1350
+Wire Wire Line
+	2850 1450 2750 1450
+Wire Wire Line
+	4000 1150 3900 1150
+Wire Wire Line
+	3900 1250 4000 1250
+Wire Wire Line
+	4000 1350 3900 1350
+Wire Wire Line
+	3900 1450 4000 1450
+Wire Wire Line
+	4000 2150 3900 2150
+Wire Wire Line
+	3900 2250 4000 2250
+Wire Wire Line
+	4000 2350 3900 2350
+Wire Wire Line
+	5150 2350 5050 2350
+Wire Wire Line
+	5050 2250 5150 2250
+Wire Wire Line
+	5150 2150 5050 2150
+Wire Wire Line
+	5050 1450 5150 1450
+Wire Wire Line
+	5150 1350 5050 1350
+Wire Wire Line
+	5050 1250 5150 1250
+Wire Wire Line
+	5150 1150 5050 1150
+Wire Wire Line
+	6300 1150 6200 1150
+Wire Wire Line
+	6200 1250 6300 1250
+Wire Wire Line
+	6300 1350 6200 1350
+Wire Wire Line
+	6200 1450 6300 1450
+Wire Wire Line
+	6300 2150 6200 2150
+Wire Wire Line
+	6200 2250 6300 2250
+Wire Wire Line
+	6300 2350 6200 2350
 $EndSCHEMATC

Commit message: Production files
Parts:
- J1, J2, J3, J4: DigikeyNumber (none) -> 732-5354-ND; ManufacturerName (none) -> Wurth Electronics Inc.; ManufacturerNumber (none) -> 61301221021
- P1: DigikeyNumber (none) -> S9175-ND; ManufacturerName (none) -> Sullins Connector Solutions; ManufacturerNumber (none) -> SBH11-PBPC-D20-ST-BK
- P2: DigikeyNumber (none) -> 732-5316-ND; ManufacturerName (none) -> Wurth Electronics; ManufacturerNumber (none) -> 61300311121
- P3: DigikeyNumber (none) -> 609-3234-ND; ManufacturerName (none) -> Amphenol FCI; ManufacturerNumber (none) -> 67997-206HLF
Changed lines of the file:
@@
 F 2 "Digilent:PMOD_DOUBLE_MALE" H 1100 1300 60  0001 C CNN
 F 3 "" H 1100 1300 60  0000 C CNN
+F 4 "61301221021" H 2500 1300 60  0001 C CNN "ManufacturerNumber"
+F 5 "732-5354-ND" H 2500 1300 60  0001 C CNN "DigikeyNumber"
+F 6 "Wurth Electronics Inc." H 2500 1300 60  0001 C CNN "ManufacturerName"
 	1    950  1300
 	1    0    0    -1
@@
 F 2 "Digilent:PMOD_DOUBLE_MALE" H 2650 1300 60  0001 C CNN
 F 3 "" H 2650 1300 60  0000 C CNN
+F 4 "61301221021" H 2500 1300 60  0001 C CNN "ManufacturerNumber"
+F 5 "732-5354-ND" H 2500 1300 60  0001 C CNN "DigikeyNumber"
+F 6 "Wurth Electronics Inc." H 2500 1300 60  0001 C CNN "ManufacturerName"
 	2    2500 1300
 	1    0    0    -1
@@
 F 2 "Digilent:PMOD_DOUBLE_MALE" H 2650 2250 60  0001 C CNN
 F 3 "" H 2650 2250 60  0000 C CNN
+F 4 "61301221021" H 2500 1300 60  0001 C CNN "ManufacturerNumber"
+F 5 "732-5354-ND" H 2500 1300 60  0001 C CNN "DigikeyNumber"
+F 6 "Wurth Electronics Inc." H 2500 1300 60  0001 C CNN "ManufacturerName"
 	3    2500 2250
 	1    0    0    -1
@@
 F 2 "Digilent:PMOD_DOUBLE_MALE" H 1100 2300 60  0001 C CNN
 F 3 "" H 1100 2300 60  0000 C CNN
+F 4 "61301221021" H 2500 1300 60  0001 C CNN "ManufacturerNumber"
+F 5 "732-5354-ND" H 2500 1300 60  0001 C CNN "DigikeyNumber"
+F 6 "Wurth Electronics Inc." H 2500 1300 60  0001 C CNN "ManufacturerName"
 	1    950  2300
 	1    0    0    -1
@@
 F 2 "Digilent:PMOD_DOUBLE_MALE" H 3800 1300 60  0001 C CNN
 F 3 "" H 3800 1300 60  0000 C CNN
+F 4 "61301221021" H 3650 1300 60  0001 C CNN "ManufacturerNumber"
+F 5 "732-5354-ND" H 3650 1300 60  0001 C CNN "DigikeyNumber"
+F 6 "Wurth Electronics Inc." H 3650 1300 60  0001 C CNN "ManufacturerName"
 	2    3650 1300
 	1    0    0    -1
@@
 F 2 "Digilent:PMOD_DOUBLE_MALE" H 3800 2300 60  0001 C CNN
 F 3 "" H 3800 2300 60  0000 C CNN
+F 4 "61301221021" H 2500 1300 60  0001 C CNN "ManufacturerNumber"
+F 5 "732-5354-ND" H 2500 1300 60  0001 C CNN "DigikeyNumber"
+F 6 "Wurth Electronics Inc." H 2500 1300 60  0001 C CNN "ManufacturerName"
 	3    3650 2300
 	1    0    0    -1
@@
 F 2 "Digilent:PMOD_DOUBLE_MALE" H 1100 3300 60  0001 C CNN
 F 3 "" H 1100 3300 60  0000 C CNN
+F 4 "61301221021" H 2500 1300 60  0001 C CNN "ManufacturerNumber"
+F 5 "732-5354-ND" H 2500 1300 60  0001 C CNN "DigikeyNumber"
+F 6 "Wurth Electronics Inc." H 2500 1300 60  0001 C CNN "ManufacturerName"
 	1    950  3300
 	1    0    0    -1
@@
 F 2 "Digilent:PMOD_DOUBLE_MALE" H 4950 1300 60  0001 C CNN
 F 3 "" H 4950 1300 60  0000 C CNN
+F 4 "61301221021" H 4800 1300 60  0001 C CNN "ManufacturerNumber"
+F 5 "732-5354-ND" H 4800 1300 60  0001 C CNN "DigikeyNumber"
+F 6 "Wurth Electronics Inc." H 4800 1300 60  0001 C CNN "ManufacturerName"
 	2    4800 1300
 	1    0    0    -1
@@
 F 2 "Digilent:PMOD_DOUBLE_MALE" H 4950 2300 60  0001 C CNN
 F 3 "" H 4950 2300 60  0000 C CNN
+F 4 "61301221021" H 2500 1300 60  0001 C CNN "ManufacturerNumber"
+F 5 "732-5354-ND" H 2500 1300 60  0001 C CNN "DigikeyNumber"
+F 6 "Wurth Electronics Inc." H 2500 1300 60  0001 C CNN "ManufacturerName"
 	3    4800 2300
 	1    0    0    -1
@@
 F 2 "Digilent:PMOD_DOUBLE_MALE" H 1100 4250 60  0001 C CNN
 F 3 "" H 1100 4250 60  0000 C CNN
+F 4 "61301221021" H 2500 1300 60  0001 C CNN "ManufacturerNumber"
+F 5 "732-5354-ND" H 2500 1300 60  0001 C CNN "DigikeyNumber"
+F 6 "Wurth Electronics Inc." H 2500 1300 60  0001 C CNN "ManufacturerName"
 	1    950  4250
 	1    0    0    -1
@@
 F 2 "Digilent:PMOD_DOUBLE_MALE" H 6100 1300 60  0001 C CNN
 F 3 "" H 6100 1300 60  0000 C CNN
+F 4 "61301221021" H 5950 1300 60  0001 C CNN "ManufacturerNumber"
+F 5 "732-5354-ND" H 5950 1300 60  0001 C CNN "DigikeyNumber"
+F 6 "Wurth Electronics Inc." H 5950 1300 60  0001 C CNN "ManufacturerName"
 	2    5950 1300
 	1    0    0    -1
@@
 F 2 "Digilent:PMOD_DOUBLE_MALE" H 6100 2300 60  0001 C CNN
 F 3 "" H 6100 2300 60  0000 C CNN
+F 4 "61301221021" H 2500 1300 60  0001 C CNN "ManufacturerNumber"
+F 5 "732-5354-ND" H 2500 1300 60  0001 C CNN "DigikeyNumber"
+F 6 "Wurth Electronics Inc." H 2500 1300 60  0001 C CNN "ManufacturerName"
 	3    5950 2300
 	1    0    0    -1
@@
 F 2 "Connectors:CONN_2.54mm_2x20" H 8100 1250 60  0001 C CNN
 F 3 "" H 8100 1250 60  0000 C CNN
+F 4 "SBH11-PBPC-D20-ST-BK" H 8100 1850 60  0001 C CNN "ManufacturerNumber"
+F 5 "S9175-ND" H 8100 1850 60  0001 C CNN "DigikeyNumber"
+F 6 "Sullins Connector Solutions" H 8100 1850 60  0001 C CNN "ManufacturerName"
 	1    8100 1850
 	1    0    0    -1
@@
 F 2 "Connectors:CONN_2.54mm_2x20" H 8100 3000 60  0001 C CNN
 F 3 "" H 8100 3000 60  0000 C CNN
+F 4 "SBH11-PBPC-D20-ST-BK" H 8100 1850 60  0001 C CNN "ManufacturerNumber"
+F 5 "S9175-ND" H 8100 1850 60  0001 C CNN "DigikeyNumber"
+F 6 "Sullins Connector Solutions" H 8100 1850 60  0001 C CNN "ManufacturerName"
 	2    8100 3600
 	1    0    0    -1
@@
 F 2 "Connectors:CONN_2.54mm_2x20" H 9550 1300 60  0001 C CNN
 F 3 "" H 9550 1300 60  0000 C CNN
+F 4 "SBH11-PBPC-D20-ST-BK" H 8100 1850 60  0001 C CNN "ManufacturerNumber"
+F 5 "S9175-ND" H 8100 1850 60  0001 C CNN "DigikeyNumber"
+F 6 "Sullins Connector Solutions" H 8100 1850 60  0001 C CNN "ManufacturerName"
 	3    9550 1900
 	1    0    0    -1
@@
 F 2 "Connectors:CONN_2.54mm_2x20" H 9550 3050 60  0001 C CNN
 F 3 "" H 9550 3050 60  0000 C CNN
+F 4 "SBH11-PBPC-D20-ST-BK" H 8100 1850 60  0001 C CNN "ManufacturerNumber"
+F 5 "S9175-ND" H 8100 1850 60  0001 C CNN "DigikeyNumber"
+F 6 "Sullins Connector Solutions" H 8100 1850 60  0001 C CNN "ManufacturerName"
 	4    9550 3650
 	1    0    0    -1
@@
 F 2 "Connectors:CONN_2.54mm_1x03" H 850 5650 60  0001 C CNN
 F 3 "" H 850 5650 60  0000 C CNN
+F 4 "61300311121" H 850 5650 60  0001 C CNN "ManufacturerNumber"
+F 5 "732-5316-ND" H 850 5650 60  0001 C CNN "DigikeyNumber"
+F 6 "Wurth Electronics" H 850 5650 60  0001 C CNN "ManufacturerName"
 	1    850  5650
 	1    0    0    -1
@@
 F 2 "Connectors:CONN_2.54mm_2x03" H 2500 5450 60  0001 C CNN
 F 3 "" H 2500 5450 60  0000 C CNN
+F 4 "67997-206HLF" H 2500 5400 60  0001 C CNN "ManufacturerNumber"
+F 5 "609-3234-ND" H 2500 5400 60  0001 C CNN "DigikeyNumber"
+F 6 "Amphenol FCI" H 2500 5400 60  0001 C CNN "ManufacturerName"
 	1    2500 5400
 	1    0    0    -1
